File: pcb/fanatone-adc2.sch (EAGLE design)
At the start: 71 parts, among them IC1 OPA2134U, IC2 DIT4192-H, IC3 PCM4201-TSSOP-16, IC4 OPA2134U, Q1 SST5484, U1 OPA1612AID, U2 TPS62240DRVTG4

Commit message: Dickson charge pump layout, PCB wip, tidy up
Parts:
- removed C31: 0.1uF, SparkFun-Capacitors:0.1UF-16V(+-10%)(0402)
- added C33: 1uF, SparkFun-Passives:CAP0805
- added D17: PMEG4005EJ, SparkFun-DiscreteSemi:DIODESOD523
- added R10: 24k9, SparkFun-Passives:RESISTOR0603-RES
- added R9: 1M, SparkFun-Passives:RESISTOR0603-RES
- C22: value 1uF -> 1uF 16V
- C23: value 4.7uF 63V -> 4.7uF 16V
- D10, D11, D12, D13, D14, D15, D4, D5, D6, D7, D8, D9: device SparkFun-DiscreteSemi:DIODE-SCHOTTKY-PMEG4005EJ -> SparkFun-DiscreteSemi:DIODESOD523
- L1: value 4.7uH -> 1uH
Connections:
- removed net N$35: C30.1, U$5.OUT
- new net N$32: C29.1, D15.C, D17.A
- net GND: now also C32.2, C33.2, R10.1
- net N$34: now also R10.2, R9.1, U$5.FB; no longer U$5.IN
- net N$38: now also D16.C
- net N$49: now also C33.1, D17.C, U$5.IN; no longer C29.1, D15.C
- net VCAPSULE-RAW: now also C30.1, R9.2, U$5.OUT
- net VDPP: now also D16.A
Other:
- note added: "5V input"
- note added: "60V - 12 * Vf_D = 57.6V 60V - 6 * Vf_D = 58.8V 72V - 6 * Vf_D = 70.8V"
- note added: "ADC SPDIF/AES3 Encoding AES42 DPP Extraction"
- note added: "Analog Input Buffer Gain Stage"
- note added: "Capsule Bias Voltage (Charge Pump) 24...80V"
- note added: "Capsule Bias Voltage 50V Boost Converter"
- note added: "GND"
- note added: "R9 = R10 ( Vout/Vref - 1 ) Vout = VCAPSULE_RAW Vref = ~1.173 (1.161...1.185) Feedback loop needs at least 10µA to be stable. I_R10 = 50µA > 10µA"
- note added: "max output voltage at 5V input: 10V input: 12V input:"
- moved on the sheet: C1, C16, C18, C2, C21, C22, C24, C25, C26, C27, C28, C29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
